File: Project-Supernova-PCB/Project-Supernova-PCB.kicad_pcb (KiCad board)
At the start: 2 copper layers, 32 parts, among them J1 Conn_01x04, J101 100k_Thermistor, J102 100k_Thermistor, J103 Screw_Terminal_01x02, J104 Conn_01x02, J105 Conn_01x02, J106 Screw_Terminal_01x02, J107 Conn_Coaxial, J108 Conn_01x04, J109 Screw_Terminal_01x02, Q101 Si1470DH, SW1 SW_SPDT, U1 S09, U101 BMP280-Module, U102 GY-NEO6MV2-Module, U103 LoRa-E5, U2 ESP32-Module-30Pin, U3 LM335D

Commit message: More work
Parts:
- removed J109: Screw_Terminal_01x02, TerminalBlock:TerminalBlock_bornier-2_P5.08mm
- removed Q101: Si1470DH, Package_TO_SOT_SMD:SOT-363_SC-70-6
- removed R2: 4.7k, Resistor_SMD:R_1206_3216Metric_Pad1.30x1.75mm_HandSolder
- added J2: Screw_Terminal_01x02, TerminalBlock:TerminalBlock_bornier-2_P5.08mm, F.Cu at (180.4, 94.2)
- added J3: Conn_01x02, Connector_PinHeader_2.54mm:PinHeader_1x02_P2.54mm_Vertical, F.Cu at (191.0, 96.5)
- added J4: Screw_Terminal_01x02, TerminalBlock:TerminalBlock_bornier-2_P5.08mm, F.Cu at (219.5, 133.6)
- added Q1: AO3420, Package_TO_SOT_SMD:SOT-23, F.Cu at (213.9, 133.6)
- added SW2: SW_SPDT, Button_Switch_THT:SW_Slide_1P2T_CK_OS102011MS2Q, F.Cu at (218.0, 93.5)
- R103: value 100k -> 10k
- R104: value 10k -> 4.7k
- U103: footprint Project-Supernova-Footprint-Lib:LoRa-E5 -> Project-Supernova-Footprint-Lib:LoRa-E5_HandSolder
- moved J107 115.0 mm to (168.5, 33.3), turned to 180 degrees
- moved C105 100.2 mm to (162.3, 38.0), turned to -90 degrees
- moved C103 98.9 mm to (137.1, 29.0), turned to 180 degrees
- moved U103 98.6 mm to (148.2, 31.2)
- moved J108 96.2 mm to (73.2, 136.1)
- moved C104 95.9 mm to (158.2, 38.0), turned to -90 degrees
- moved C1 91.3 mm to (137.1, 26.4), turned to 180 degrees
- moved R104 90.1 mm to (207.8, 76.4)
- moved R103 90.1 mm to (207.8, 73.2)
- moved L101 86.2 mm to (160.0, 33.5)
- moved C106 67.5 mm to (68.0, 136.7)
- moved J104 65.7 mm to (211.6, 83.3)
- moved U102 65.1 mm to (80.8, 78.7), turned to -90 degrees
- moved C101 64.8 mm to (193.5, 149.9)
- moved J1 62.7 mm to (142.2, 42.7), turned to 90 degrees
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Connections:
- net Net-(U3-V+) renamed TEMP_SENSE_ONBOARD
- R1 pad 1: unconnected-(R1-Pad1) -> +3V3
- U101 pad 3: unconnected-(U101-SCL-Pad3) -> SCL
- U101 pad 4: SCL -> SDA
- U102 pad 2: GPS_MOSI -> GPS_UART_MOSI
- U102 pad 3: GPS_MISO -> GPS_UART_MISO
- U2 pad 1: unconnected-(U2-3V3-Pad1) -> +3V3
- U2 pad 2: unconnected-(U2-GND_2-Pad2) -> GND
- U2 pad 29: unconnected-(U2-GND_1-Pad29) -> GND
- U2 pad 30: unconnected-(U2-VIN-Pad30) -> MCU_VIN
- U2 pad 6: LORA_UART_MISO -> unconnected-(U2-RX2/D16-Pad6)
- U2 pad 7: LORA_UART_MOSI -> unconnected-(U2-TX2/D17-Pad7)
Other:
- board text added: "3V3"
- board text added: "GND"
- board text added: "RX"
- board text added: "TX"
- board text added: "To Heater"

Commit message: Lay out PCB
Parts:
- added H1: MountingHole_Pad, MountingHole:MountingHole_3.2mm_M3_DIN965_Pad, F.Cu at (180.3, 49.5)
- added H2: MountingHole_Pad, MountingHole:MountingHole_3.2mm_M3_DIN965_Pad, F.Cu at (88.9, 49.5)
- added H3: MountingHole_Pad, MountingHole:MountingHole_3.2mm_M3_DIN965_Pad, F.Cu at (180.3, 129.5)
- added H4: MountingHole_Pad, MountingHole:MountingHole_3.2mm_M3_DIN965_Pad, F.Cu at (88.9, 129.5)
- moved J11 129.4 mm to (96.5, 125.7)
- moved J9 118.7 mm to (97.8, 116.8), turned to 90 degrees
- moved SW2 107.0 mm to (120.7, 128.0), turned to 90 degrees
- moved SW1 96.1 mm to (128.3, 128.0), turned to 90 degrees
- moved J3 92.3 mm to (99.1, 104.1)
- moved J6 83.8 mm to (135.9, 127.0)
- moved U2 80.0 mm to (166.4, 72.4)
- moved Q1 77.3 mm to (138.8, 115.6)
- moved J10 76.4 mm to (110.5, 116.8), turned to 90 degrees
- moved J12 74.4 mm to (109.2, 125.7)
- moved R4 57.6 mm to (160.0, 105.4)
- moved J4 55.5 mm to (116.3, 52.1), turned to 0 degrees
- moved C6 55.4 mm to (168.9, 100.3)
- moved R2 55.4 mm to (168.9, 104.3)
- moved J5 55.4 mm to (173.5, 100.8)
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- renumbered C106 to C2, C103 to C3, C104 to C4, C105 to C5, C101 to C6, C102 to C7, J105 to J10, J103 to J11, J106 to J12, J108 to J2, J107 to J4, J101 to J5, J4 to J6, J2 to J7, J102 to J8, J104 to J9, L101 to L1, R101 to R2, R102 to R3, R103 to R4, R104 to R5, SW2 to SW1, SW1 to SW2, U102 to U1, U101 to U2, U103 to U3, U3 to U4, U2 to U5, U1 to U6
Connections:
- SW1 pad 2: GND -> RTF_SWITCH
- U5 pad 11: unconnected-(U2-D21/I2C_SDA-Pad11) -> SDA
- U5 pad 14: unconnected-(U2-D22/I2C_SCL-Pad14) -> SCL
- U5 pad 19: unconnected-(U2-D34/ADC1_CH6-Pad19) -> TEMP_SENSE_ONBOARD
- U5 pad 20: unconnected-(U2-D35/ADC1_CH7-Pad20) -> TEMP_V+
- U5 pad 21: unconnected-(U2-D32/ADC1_CH4/TOUCH9-Pad21) -> TEMP_SENSE_2
- U5 pad 22: unconnected-(U2-D33/ADC1_CH5/TOUCH8-Pad22) -> TEMP_SENSE_1
- U5 pad 25: unconnected-(U2-D27/ADC2_CH7/TOUCH7-Pad25) -> BATT_SENSE
- U5 pad 26: unconnected-(U2-D14/ADC2_CH6/TOUCH6/HSPI_CLK-Pad26) -> HEATER_EN
- U5 pad 27: unconnected-(U2-D12/ADC2_CH5/TOUCH5/HSPI_MISO-Pad27) -> DHT_DATA
- U5 pad 4: unconnected-(U2-D2/ADC2_CH2/TOUCH2-Pad4) -> GPS_UART_MOSI
- U5 pad 5: unconnected-(U2-D4/ADC2_CH0/TOUCH0-Pad5) -> GPS_UART_MOSI
- U5 pad 6: unconnected-(U2-RX2/D16-Pad6) -> LORA_UART_MISO
- U5 pad 7: unconnected-(U2-TX2/D17-Pad7) -> LORA_UART_MOSI
- U5 pad 9: unconnected-(U2-D18/VSPI_CLK-Pad9) -> RTF_SWITCH
Other:
- board outline added: 99.1 x 87.6 mm
- board text added: "GND|3V3"
- board text added: "GND|BATT"
- board text added: "GND|uC_VIN"

Commit message: Routed PCB
Parts:
- moved C3 33.5 mm to (117.1, 69.6), turned to 90 degrees
- moved C1 29.7 mm to (120.0, 69.6), turned to 90 degrees
- moved C4 29.4 mm to (98.9, 58.7)
- moved L1 29.3 mm to (97.4, 63.5)
- moved J1 28.7 mm to (166.8, 55.6)
- moved C5 28.6 mm to (95.8, 58.7)
- moved J4 26.6 mm to (91.1, 60.8)
- moved U3 5.34 mm to (107.7, 67.6)
- moved J12 0.64 mm to (108.6, 125.7)
Connections:
- U5 pad 5: GPS_UART_MOSI -> GPS_UART_MISO
Routing:
- net DHT_DATA: track 0.00 -> 89.1 mm, vias 0 -> 1
- net LORA_UART_MOSI: track 0.00 -> 85.1 mm, vias 0 -> 1
- net LORA_UART_MISO: track 0.00 -> 83.9 mm, vias 0 -> 1
- net +BATT: track 0.00 -> 69.3 mm
- net SCL: track 0.00 -> 64.7 mm, vias 0 -> 1
- net MCU_VIN: track 0.00 -> 60.7 mm
- net GPS_UART_MOSI: track 0.00 -> 54.3 mm, vias 0 -> 1
- net SDA: track 0.00 -> 50.4 mm, vias 0 -> 1
- net GPS_UART_MISO: track 0.00 -> 48.3 mm, vias 0 -> 2
- net BATT_SENSE: track 0.00 -> 45.7 mm, vias 0 -> 1
- net RTF_SWITCH: track 0.00 -> 41.9 mm, vias 0 -> 1
- net HEATER_EN: track 0.00 -> 41.3 mm, vias 0 -> 1
- net TEMP_SENSE_1: track 0.00 -> 31.7 mm, vias 0 -> 2
- net Net-(J11-Pin_2): track 0.00 -> 30.1 mm
- net TEMP_SENSE_2: track 0.00 -> 26.6 mm
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- added copper zone on B.Cu, net +3V3
- added copper zone on B.Cu, net GND
- added copper zone on F.Cu, net GND
- added copper zone on F.Cu, net Net-(U3-RFIO)
Other:
- board text added: "DHT_DATA"
- board text added: "GPS_MISO"
- board text added: "GPS_MOSI"
- board text added: "OFF | ON (PWR)"
- board text added: "REV 1 2023-05-19 Balloon Pals"
- board text added: "SIT | FLY (RTF)"
- board text added: "TEMP SENSE 1"
- board text added: "TEMP SENSE 2"
- board text added: "X"
