File: Project-Supernova-PCB/Project-Supernova-PCB.kicad_sch (KiCad schematic)
At the start: 38 parts, among them J1 Conn_01x04, J10 Conn_01x02, J11 Screw_Terminal_01x02, J12 Screw_Terminal_01x02, J2 Conn_01x04, J3 Conn_01x02, J4 Conn_Coaxial, J6 100k_Thermistor, J6 Screw_Terminal_01x02, J7 100k_Thermistor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

Commit message: PCB changes, finish Rev1 as ordered
Parts:
- added D1, D2, D3: LED, LED_SMD:LED_1206_3216Metric_Pad1.42x1.75mm_HandSolder, symbol Device:LED
- added H5, H6: MountingHole, MountingHole:MountingHole_3mm, symbol Mechanical:MountingHole
- added J13: Conn_01x03, Connector_PinHeader_2.54mm:PinHeader_1x03_P2.54mm_Vertical, symbol Connector_Generic:Conn_01x03
- added R10: 3.3k, Resistor_SMD:R_1206_3216Metric_Pad1.30x1.75mm_HandSolder, symbol Device:R
- added R6, R7: 4.7k, Resistor_SMD:R_1206_3216Metric_Pad1.30x1.75mm_HandSolder, symbol Device:R
- added R8, R9: 1k, Resistor_SMD:R_1206_3216Metric_Pad1.30x1.75mm_HandSolder, symbol Device:R
- added TP1: TestPoint, TestPoint:TestPoint_Pad_D3.0mm, symbol Connector:TestPoint
- added TP2, TP3: TestPoint, TestPoint:TestPoint_Pad_D4.0mm, symbol Connector:TestPoint
- J4: footprint Connector_Coaxial:SMA_Molex_73251-1153_EdgeMount_Horizontal -> Connector_Coaxial:SMA_Wurth_60312002114503_Vertical
- U5: symbol Project-Supernova-Symbol-Lib:ESP32-Module -> Project-Supernova-Symbol-Lib:ESP32-Module-30Pin
Connections:
- net +3V3: now also R6.1, R7.1, R9.1
- net +BATT: now also R10.1
- net GND: now also D1.1 (K), D2.1 (K), D3.1 (K)
- net SCL: now also R7.2
- net SDA: now also R6.2
- net at U5.15 (D23/VSPI_MOSI): now also J13.1 (Pin_1)
- net at U5.23 (D25/ADC2_CH8/DAC1): now also J13.2 (Pin_2)
- net at U5.24 (D26/ADC2_CH9/DAC2): now also J13.3 (Pin_3)
- net TOUCH4: now reaches U5.28 (D13/ADC2_CH4/TOUCH4/HSPI_MOSI)
- net TOUCH4: now also TP2.1
- net TOUCH3: now reaches U5.3 (D15/ADC2_CH3/TOUCH3/HSPI_CS0)
- net TOUCH3: now also TP3.1
- net at U5.8 (D5/VSPI_CS0): now also R8.1
- net at U3.28 (PB0): now also TP1.1
- new net: D2.2 (A), R9.2
- new net: D3.2 (A), R10.2
- new net: D1.2 (A), R8.2
- no-connect marks 37 -> 30
Other:
- note added: "GP Breakout"
- note added: "I2C Pullups"
- note added: "Unknown TP purpose It's on the ref. schematic though"
- moved on the sheet: C2, H2, H3, H4, J2, J3, R4, R5, SW1, U1

Commit message: Add Rev1.1 hot fix notes
Parts:
- C4, C5, R2, U4: now not fitted
- R4: value 10k -> 18k
Connections:
- net DHT_DATA: now also J13.1 (Pin_1), U5.15 (D23/VSPI_MOSI); no longer U5.27 (D12/ADC2_CH5/TOUCH5/HSPI_MISO)
- net TEMP_V+: now also J13.2 (Pin_2), U5.23 (D25/ADC2_CH8/DAC1)
- no-connect marks 30 -> 31
Other:
- note added: "Active High Drive"
- note added: "Divider Ratio: 4.7k/22.7k = 0.207048x 12V battery/supply turns into 2.48V max"
- note added: "ERRATA: Onboard Temp Sensor is useless"
- note added: "Formerly DHT_DATA on D12"
- note added: "Moved"
- note added: "To Heater (7.8 ohms)"
- note removed: "Divider Ratio: 4.7k/14.7k = 0.3197x 10V battery turns into 3.2V max"
- note removed: "Probably active high lol?"
- note removed: "To Heater"
Changed lines of the file:
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@@
 (kicad_sch (version 20230121) (generator eeschema)
   (paper "USLetter")
+  (junction (at 176.53 78.74) (diameter 0) (color 0 0 0 0)
+  )
   (junction (at 96.52 45.72) (diameter 0) (color 0 0 0 0)
   )
@@
   (junction (at 36.83 82.55) (diameter 0) (color 0 0 0 0)
   )
+  (junction (at 176.53 81.28) (diameter 0) (color 0 0 0 0)
+  )
   (junction (at 231.14 160.02) (diameter 0) (color 0 0 0 0)
   )
@@
   (no_connect (at 86.36 149.86))
   (no_connect (at 228.6 124.46))
+  (no_connect (at 111.76 100.33))
   (no_connect (at 50.8 165.1))
   (no_connect (at 50.8 160.02))
@@
     (stroke (width 0) (type default))
   )
+  (wire (pts (xy 176.53 78.74) (xy 191.77 78.74))
+    (stroke (width 0) (type default))
+  )
   (wire (pts (xy 45.72 35.56) (xy 49.53 35.56))
     (stroke (width 0) (type default))
@@
     (stroke (width 0) (type default))
   )
+  (wire (pts (xy 176.53 81.28) (xy 191.77 81.28))
+    (stroke (width 0) (type default))
+  )
   (wire (pts (xy 215.9 87.63) (xy 215.9 92.71))
     (stroke (width 0) (type default))
@@
     (stroke (width 0) (type default))
   )
-  (text "To Heater" (at 170.18 144.78 0)
+  (text "To Heater\n(7.8 ohms)" (at 168.91 139.7 0)
     (effects (font (size 1.27 1.27)) (justify left bottom))
   )
@@
     (effects (font (size 1.27 1.27)) (justify left bottom))
   )
+  (text "ERRATA: Onboard Temp Sensor is useless" (at 121.92 21.59 0)
+    (effects (font (size 1.27 1.27)) (justify left bottom))
+  )
   (text "Ready to Fly Switch" (at 212.09 105.41 90)
     (effects (font (size 2 2) (thickness 0.4) bold) (justify left bottom))
@@
     (effects (font (size 2 2) (thickness 0.4) bold) (justify left bottom))
   )
+  (text "Formerly DHT_DATA on D12" (at 120.65 100.33 0)
+    (effects (font (size 1.27 1.27)) (justify right bottom))
+  )
   (text "To DHT22" (at 49.53 91.44 0)
     (effects (font (size 1.27 1.27)) (justify left bottom))
   )
-  (text "Divider Ratio: 4.7k/14.7k = 0.3197x\n10V battery turns into 3.2V max"
-    (at 229.87 106.68 0)
+  (text "Moved" (at 179.07 97.79 0)
+    (effects (font (size 1.27 1.27)) (justify left bottom))
+  )
+  (text "Divider Ratio: 4.7k/22.7k = 0.207048x\n12V battery/supply turns into 2.48V max"
+    (at 226.06 106.68 0)
     (effects (font (size 1.27 1.27)) (justify left bottom))
   )
-  (text "Probably active high lol?" (at 133.35 156.21 0)
+  (text "Active High Drive" (at 133.35 156.21 0)
     (effects (font (size 1.27 1.27)) (justify left bottom))
   )
@@
     )
   )
+  (global_label "TEMP_V+" (shape input) (at 184.15 96.52 0) (fields_autoplaced)
+    (effects (font (size 1.27 1.27)) (justify left))
+    (property "Intersheetrefs" "${INTERSHEET_REFS}" (at 195.5224 96.52 0)
+      (effects (font (size 1.27 1.27)) (justify left) hide)
+    )
+  )
   (global_label "LORA_UART_MISO" (shape input) (at 62.23 182.88 180) (fields_autoplaced)
     (effects (font (size 1.27 1.27)) (justify right))
@@
     )
   )
+  (global_label "DHT_DATA" (shape input) (at 191.77 78.74 0) (fields_autoplaced)
+    (effects (font (size 1.27 1.27)) (justify left))
+    (property "Intersheetrefs" "${INTERSHEET_REFS}" (at 203.6263 78.74 0)
+      (effects (font (size 1.27 1.27)) (justify left) hide)
+    )
+  )
   (global_label "LORA_UART_MOSI" (shape input) (at 107.95 87.63 180) (fields_autoplaced)
     (effects (font (size 1.27 1.27)) (justify right))
@@
     )
   )
-  (global_label "TEMP_V+" (shape input) (at 184.15 96.52 0) (fields_autoplaced)
+  (global_label "TEMP_V+" (shape input) (at 191.77 81.28 0) (fields_autoplaced)
     (effects (font (size 1.27 1.27)) (justify left))
-    (property "Intersheetrefs" "${INTERSHEET_REFS}" (at 195.5224 96.52 0)
+    (property "Intersheetrefs" "${INTERSHEET_REFS}" (at 203.1424 81.28 0)
       (effects (font (size 1.27 1.27)) (justify left) hide)
     )
@@
     )
   )
-  (global_label "DHT_DATA" (shape input) (at 111.76 100.33 180) (fields_autoplaced)
-    (effects (font (size 1.27 1.27)) (justify right))
-    (property "Intersheetrefs" "${INTERSHEET_REFS}" (at 99.9037 100.33 0)
-      (effects (font (size 1.27 1.27)) (justify right) hide)
-    )
-  )
   (global_label "SCL" (shape input) (at 45.72 35.56 180) (fields_autoplaced)
     (effects (font (size 1.27 1.27)) (justify right))
@@
   )
   (symbol (lib_id "Device:C") (at 114.3 171.45 0) (mirror y) (unit 1)
-    (in_bom yes) (on_board yes) (dnp no)
+    (in_bom yes) (on_board yes) (dnp yes)
     (property "Reference" "C5" (at 111.76 170.18 0)
       (effects (font (size 1.27 1.27)) (justify left))
@@
   (symbol (lib_id "Device:R") (at 233.68 78.74 0) (unit 1)
     (in_bom yes) (on_board yes) (dnp no) (fields_autoplaced)
-    (property "Reference" "R4" (at 236.22 78.105 0)
+    (property "Reference" "R4" (at 236.22 77.47 0)
       (effects (font (size 1.27 1.27)) (justify left))
     )
-    (property "Value" "10k" (at 236.22 80.645 0)
+    (property "Value" "18k" (at 236.22 80.01 0)
       (effects (font (size 1.27 1.27)) (justify left))
     )
@@
   )
   (symbol (lib_id "Device:C") (at 100.33 171.45 0) (mirror y) (unit 1)
-    (in_bom yes) (on_board yes) (dnp no)
+    (in_bom yes) (on_board yes) (dnp yes)
     (property "Reference" "C4" (at 97.79 170.18 0)
       (effects (font (size 1.27 1.27)) (justify left))
@@
   )
   (symbol (lib_id "power:GND") (at 148.59 48.26 0) (unit 1)
-    (in_bom yes) (on_board yes) (dnp no)
+    (in_bom yes) (on_board yes) (dnp yes)
     (property "Reference" "#PWR04" (at 148.59 54.61 0)
       (effects (font (size 1.27 1.27)) hide)
@@
   )
   (symbol (lib_id "Project-Supernova-Symbol-Lib:LM335D") (at 148.59 39.37 0) (unit 1)
-    (in_bom yes) (on_board yes) (dnp no) (fields_autoplaced)
+    (in_bom yes) (on_board yes) (dnp yes) (fields_autoplaced)
     (property "Reference" "U4" (at 152.4 38.735 0)
       (effects (font (size 1.27 1.27)) (justify left))
@@
   )
   (symbol (lib_id "Device:R") (at 148.59 25.4 0) (unit 1)
-    (in_bom yes) (on_board yes) (dnp no) (fields_autoplaced)
+    (in_bom yes) (on_board yes) (dnp yes) (fields_autoplaced)
     (property "Reference" "R2" (at 151.13 24.765 0)
       (effects (font (size 1.27 1.27)) (justify left))

Commit message: Main Rev2 schematic changes
Parts:
- removed TP2, TP3: TestPoint, TestPoint:TestPoint_Pad_D4.0mm, symbol Connector:TestPoint
- added C8: 10u, Capacitor_SMD:C_1206_3216Metric_Pad1.33x1.80mm_HandSolder, symbol Device:C
- added D4: LED, LED_SMD:LED_1206_3216Metric_Pad1.42x1.75mm_HandSolder, symbol Device:LED
- added R11: 10k, Resistor_SMD:R_1206_3216Metric_Pad1.30x1.75mm_HandSolder, symbol Device:R
- added R12: 3.3k, Resistor_SMD:R_1206_3216Metric_Pad1.30x1.75mm_HandSolder, symbol Device:R
- added R13, R14: 4.7k, Resistor_SMD:R_1206_3216Metric_Pad1.30x1.75mm_HandSolder, symbol Device:R
- added R15: 1k, Resistor_SMD:R_1206_3216Metric_Pad1.30x1.75mm_HandSolder, symbol Device:R
- R2, R3: value 4.7k -> 75k
Connections:
- net +3V3: now also R11.1, R13.1; no longer SW1.3 (C)
- net DHT_DATA: now also U5.24 (D26/ADC2_CH9/DAC2), R11.2; no longer J13.1 (Pin_1), U5.15 (D23/VSPI_MOSI)
- net GND: now also C8.2, D4.1 (K), R12.2, R14.2; no longer SW1.1 (A)
- net HEATER_EN: now also R12.1, R15.1
- net TEMP_V+: no longer J13.2 (Pin_2), U5.20 (D35/ADC1_CH7)
- net at U5.16 (EN): now also C8.1
- net at J13.3 (Pin_3): no longer U5.24 (D26/ADC2_CH9/DAC2)
- net TOUCH3: no longer names the net of U5.3 (D15/ADC2_CH3/TOUCH3/HSPI_CS0)
- net TOUCH4: no longer names the net of U5.28 (D13/ADC2_CH4/TOUCH4/HSPI_MOSI)
- new net: R14.1, SW1.1 (A)
- new net: R13.2, SW1.3 (C)
- new net: D4.2 (A), R15.2
- no-connect marks 31 -> 29
Other:
- note added: "FIXME swap out a different board temp sensor"
- note added: "TODO change GPS UART off of Pin 2 (onboard LED)"
- note added: "TODO change thermoster connector footprint to a normal pull-safe one"
- note added: "TODO vreg footprint, mosfet footprint, move pads voltage divider resistors TODO via inside pad"
- note removed: "Formerly DHT_DATA on D12"
- note removed: "Moved"
- moved on the sheet: C2, J13, J2, R4, R5

Commit message: Lock in Rev2 Gerber
Parts:
- removed J13: Conn_01x03, Connector_PinHeader_2.54mm:PinHeader_1x03_P2.54mm_Vertical, symbol Connector_Generic:Conn_01x03
- removed J3: Conn_01x02, Connector_PinHeader_2.54mm:PinHeader_1x02_P2.54mm_Vertical, symbol Connector_Generic:Conn_01x02
- removed R2: 4.7k, Resistor_SMD:R_1206_3216Metric_Pad1.30x1.75mm_HandSolder, symbol Device:R
- removed U4: LM335D, Package_SO:SOIC-8_3.9x4.9mm_P1.27mm, symbol Project-Supernova-Symbol-Lib:LM335D
- added H10, H11, H12, H7, H8, H9: MountingHole, MountingHole:MountingHole_2mm, symbol Mechanical:MountingHole
- added J13, J14, J15, J3: Conn_01x04, Connector_PinHeader_2.54mm:PinHeader_1x04_P2.54mm_Vertical, symbol Connector_Generic:Conn_01x04
- added R1: 0, Resistor_SMD:R_1206_3216Metric_Pad1.30x1.75mm_HandSolder, symbol Device:R
- added U4: STDS75DS2F, Package_SO:MSOP-8_3x3mm_P0.65mm, symbol Project-Supernova-Symbol-Lib:STDS75DS2F
- H5, H6: footprint MountingHole:MountingHole_3mm -> MountingHole:MountingHole_2mm
- Q1: footprint Package_TO_SOT_SMD:SOT-23 -> Project-Supernova-Footprint-Lib:SOT-23-MassivePads-HandSolder
Connections:
- net TEMP_SENSE_ONBOARD is gone; now on net BATT_SENSE: U5.19 (D34/ADC1_CH6)
- net +3V3: now also J14.1 (Pin_1), J14.2 (Pin_2), J14.3 (Pin_3), J14.4 (Pin_4), U4.8 (VDD)
- net +BATT: now also J13.1 (Pin_1), J13.2 (Pin_2), J13.3 (Pin_3), J13.4 (Pin_4)
- net BATT_SENSE: no longer U5.25 (D27/ADC2_CH7/TOUCH7)
- net GND: now also J15.1 (Pin_1), J15.2 (Pin_2), J15.3 (Pin_3), J15.4 (Pin_4), U4.4 (GND), U4.5 (A2), U4.6 (A1), U4.7 (A0)
- net GPS_UART_MOSI: now also U5.28 (D13/ADC2_CH4/TOUCH4/HSPI_MOSI); no longer U5.4 (D2/ADC2_CH2/TOUCH2)
- net HEATER_EN: now also R1.1; no longer Q1.1 (G), R12.1
- net SCL: now also U4.2 (SCL)
- net SDA: now also U4.1 (SDA)
- net at U5.10 (D19/VSPI_MISO): now also J3.1 (Pin_1)
- net at U5.15 (D23/VSPI_MOSI): now also J3.2 (Pin_2)
- net at U5.20 (D35/ADC1_CH7): now also J3.4 (Pin_4)
- new net: J3.3 (Pin_3), U5.25 (D27/ADC2_CH7/TOUCH7)
- new net: Q1.1 (G), R1.2, R12.1
- no-connect marks 29 -> 31
Other:
- note added: "Active High Ctrl"
- note added: "Address: 1001_A2_A1_A0_R~{W} Address: 1001_0_0_0_1 When R~{W}=1, READ mode"
- note added: "D2 = Onb. LED"
- note added: "DNU D12"
- note added: "ESP32 has internal temperature sensor, 12-bit ADC (3V3) [+/- 10% welp], but disabled on many models"
- note removed: "Active High Drive"
- note removed: "ERRATA: Onboard Temp Sensor is useless"
- note removed: "ESP32 has internal temperature sensor, 12-bit ADC (3V3) [+/- 10% welp]"
- note removed: "FIXME swap out a different board temp sensor"
- note removed: "TODO change GPS UART off of Pin 2 (onboard LED)"
- note removed: "TODO change thermoster connector footprint to a normal pull-safe one"
- note removed: "TODO vreg footprint, mosfet footprint, move pads voltage divider resistors TODO via inside pad"
- moved on the sheet: H5, H6, R12, R6, R7
